File: imu_LSM6DSL/imu_LSM6DSL.kicad_pcb (KiCad board)
At the start: 4 copper layers, 7 parts, among them J1 Conn_01x02, J2 Conn_01x06, U1 LSM6DSLTR

Commit message: Final version
Parts:
- moved R_sda1 1.83 mm to (129.9, 94.3)
- moved R_scl1 1.65 mm to (129.7, 82.0)
- moved C1 0.73 mm to (128.0, 90.4)
- moved C2 0.36 mm to (131.4, 90.3)
Routing:
- net VDDIO: track 13.2 -> 33.9 mm, vias 1 -> 3
- net GND: track 9.71 -> 21.8 mm, vias 0 -> 1
- net /SDO/SA0: track 10.9 -> 19.1 mm, vias 0 -> 1
- net /SDA: track 25.8 -> 31.7 mm
- net /INT2: track 12.9 -> 7.34 mm, vias 2 -> 1
- net (no net): track 5.50 -> 0.00 mm
- net /INT1: track 13.3 -> 18.2 mm, vias 0 -> 1
- net Net-(U1-VDD): track 7.73 -> 9.77 mm
- net /SCL: track 11.4 -> 12.2 mm, vias 3 -> 0
- net /CS: track 9.40 -> 9.71 mm, vias 0 -> 1
Other:
- board outline added: 20.6 x 18.6 mm
